Commit message: Proyecto final: costos, peso, eléctrica, LLM, PyBullet, carrusel y revisiones; READMEs de los temas 1-9
Proyecto final (pedidos del equipo para el profesor):
- Costos de la estructura 3D pieza por pieza y peso total del montaje (docs/costos.md, docs/peso.md).
- Parte eléctrica simulada punto por punto (sim/electrica.py, docs/electrica.md) y circuitos en wokwi/.
- Asistente enfocado en monedas y carro (60/60 con modelo local y reglas) y docs/modelo-local.md (Qwen2.5-3B).
- Lógica interna explicada (docs/logica-interna.md), simulaciones de PyBullet en ventana (simulaciones.bat,
  sim/ver/) con videos, y física vs 3D (docs/fisica-vs-3d.md).
- Carrusel con su tiempo real: la moneda espera a que su tubo esté quieto y termina de caer antes del
  siguiente giro (control/carrusel.py); pausa de vasos 1400 ms.
- Firmware: prensa/empujador excluyentes, PWM del carro al 70 %, I2C largo a 100 kHz, reposo del A4988,
  paro enclavado, cortina que falla del lado seguro, canaleta con puede_soltar_vaso, sesión del protocolo,
  WDT, límite de ESP-NOW.
- Dos rondas de revisión lógica y visual: asistente sin órdenes por error, puente serial con buffer,
  supervisor robusto, dashboard (matriz, cifras, 900 px, sin caídas), visor (panel, etiquetas, vistas).

Temas 1-9: READMEs reescritos (qué es, diagramas, conexiones pin a pin, qué hace cada archivo, lógica,
cómo probarlo) y arreglos: tema 4 (reglas por partes), tema 6 (pulgar, 330 ohm), comentarios de 7/8/9.

924+ pruebas en verde.

Co-Authored-By: Claude Opus 5.5 <noreply@anthropic.com>
Claude-Session: https://claude.ai/code/session_011w9mKXGscftFnQfDpWbrmg

File: proyecto-final/sim/urdf/cinta_vasos.urdf (robot description, URDF)
Before this commit: robot cinta_vasos, 4 links, 3 joints
Links:
- link bancada: geometry collision box size=0.395 0.075 0.002; collision box size=0.40 0.08 0.02
- link bandeja_rechazo_vasos: geometry collision box size=0.096 0.116 0.004; visual box size=0.096 0.116 0.004
Joints:
- joint junta_bandeja_rechazo: origin xyz=0.16 0.10 0.005 rpy=0 0 0 -> xyz=0.27 0.00 -0.098 rpy=0 0 0

Commit message: Proyecto final: carro y maqueta completa impresos en PLA, ahorro de costos y visor igual a lo físico
- chasis_impreso/: carro paramétrico en OpenSCAD con uniones a presión (remaches impresos), tandas 3MF,
  STL por pieza, revisores (voladizos, remaches medidos en el ensamble), manual con conexiones hilo por
  hilo, lista de materiales y visor del carro armado.
- maqueta_impresa/: toda la planta en PLA sin perfil 2020 (estructura de tubos 16x16 y nodos, almacén,
  cintas, tapas/prensa/empujador, canaleta y muelle). revisar.py mide cada remache, choques, barridos de
  lo que se mueve y voladizos; probar_revisor.py lo prueba con 39 errores a propósito. 2,68 kg en 25
  tandas, material.md y manual_maqueta.pdf.
- Visor 3D y simulación dibujan la maqueta impresa (maqueta_impresa.glb) con prueba de coincidencia.
- Ahorros aprobados: sin bornera, IEC, optoacopladores (M18 con BAT85 + pull-up), hub USB, reparto
  I2C, canaletas ni MDF; un fusible, fuente y buck de 5 A. Costo $1.998.921 -> $1.387.143.

Co-Authored-By: Claude Fable 5.1 <noreply@anthropic.com>

File: proyecto-final/sim/urdf/cinta_vasos.urdf (robot description, URDF)
Before this commit: robot cinta_vasos, 4 links, 3 joints
Links:
- link bancada: geometry collision box size=0.374 0.0806 0.0159; collision box size=0.395 0.075 0.002
- link empujador_descarga: geometry visual box size=0.056 0.004 0.055
Joints:
- joint junta_empujador_descarga: axis 0 0 1 -> 0 -1 0; limit lower=0 upper=1.45 effort=5 velocity=4 -> lower=0 upper=0.0675 effort=5 velocity=0.5; origin xyz=0.12 -0.04 0.032 rpy=0 0 0 -> xyz=0.16 0.045 0.0655 rpy=0 0 0; type revolute -> prismatic

Commit message: Maqueta impresa: auditoría completa, segunda opinión aplicada y 3MF con la configuración adentro
- Primera capa: la causa de alm_1 era el perfil con wipe y el filamento del sistema, más la rejilla vieja.
  Ahora cada 3MF trae el proceso y el filamento "maqueta" (exportar.py + perfil_creality.json) y
  laminar.py lamina las 26 tandas con el CLI de Creality Print y revisa cada G-code.
- Revisor: primera capa, base y despegue (primera_capa.py), sin soportes capa por capa (voladizos.py),
  auditoría por pieza (auditar.py), mecanismos fase por fase y barridos completos; 128 casos de prueba.
  Única excepción aceptada: el puente de 30 mm de la cumbrera de mon_e4 (voladizos.PUENTES_ACEPTADOS).
- Segunda opinión: sin partes que nazcan en el aire (mon_e4, tap_pre_placa, vas_lat_s_b), postes del
  NEMA con nervio, sin el rodillo de retorno C, canaleta amarrada, 11 separadores en la banda de vasos,
  obturador de corredera, precios de lo que el manual manda comprar, visor y firmware al día.
- Revisión completa en TODO OK (183 piezas, 316 remaches), auditoría sin fallas, esfuerzos cumplen,
  2,98 kg estimados (Creality Print: 2,95 kg y 101 h), costo $1.586.033, peso 8,08 kg, 950 pruebas.

Co-Authored-By: Claude Opus 5.5 <noreply@anthropic.com>

File: proyecto-final/sim/urdf/cinta_vasos.urdf (robot description, URDF)
Before this commit: robot cinta_vasos, 4 links, 3 joints
Links:
- link bancada: geometry collision box size=0.370 0.0806 0.0159; collision box size=0.395 0.075 0.002
